Commit message: feat: rm some static number

File: legged_examples/legged_unitree/legged_unitree_description/urdf/common/leg.xacro (robot description, xacro)
@@ -130,10 +130,10 @@
             </inertial>
         </link>
-        <joint name="${prefix}_foot_fixed" type="fixed" dont_collapse="true">
+        <joint name="${prefix}_FOOT_fixed" type="fixed">
             <origin rpy="0 0 0" xyz="0 0 ${-(calf_length)}"/>
             <parent link="${prefix}_calf"/>
-            <child link="${prefix}_FOOT"/>
+            <child link="${prefix}_foot"/>
         </joint>
-        <link name="${prefix}_FOOT">
+        <link name="${prefix}_foot">
             <visual>
                 <origin rpy="0 0 0" xyz="0 0 0"/>
@@ -157,5 +157,5 @@
             </inertial>
         </link>
-        <gazebo reference="${prefix}_foot_fixed">
+        <gazebo reference="${prefix}_FOOT_fixed">
             <disableFixedJointLumping>true</disableFixedJointLumping>
         </gazebo>
@@ -178,5 +178,5 @@
             <self_collide>1</self_collide>
         </gazebo>
-        <gazebo reference="${prefix}_FOOT">
+        <gazebo reference="${prefix}_foot">
             <mu1>0.6</mu1>
             <mu2>0.6</mu2>
